Commit message: fix a1 model

File: assets/a1_description/a1.urdf (robot description, URDF)
Before this commit: robot a1_description, 18 links, 17 joints
Joints:
- joint FL_hip_joint: limit lower=-0.802851455917 upper=0.802851455917 -> lower=-1.4 upper=1.4; type continuous -> revolute
- joint FL_lower_joint: limit lower=-2.69653369433 upper=-0.916297857297 -> lower=0.916297857297 upper=2.69653369433; type continuous -> revolute
- joint FR_hip_joint: limit lower=-0.802851455917 upper=0.802851455917 -> lower=-1.4 upper=1.4; type continuous -> revolute
- joint FR_lower_joint: limit lower=-2.69653369433 upper=-0.916297857297 -> lower=0.916297857297 upper=2.69653369433; type continuous -> revolute
- joint RL_hip_joint: limit lower=-0.802851455917 upper=0.802851455917 -> lower=-1.4 upper=1.4; type continuous -> revolute
- joint RL_lower_joint: limit lower=-2.69653369433 upper=-0.916297857297 -> lower=0.916297857297 upper=2.69653369433; type continuous -> revolute
- joint RR_hip_joint: limit lower=-0.802851455917 upper=0.802851455917 -> lower=-1.4 upper=1.4; type continuous -> revolute
- joint RR_lower_joint: limit lower=-2.69653369433 upper=-0.916297857297 -> lower=0.916297857297 upper=2.69653369433; type continuous -> revolute
