Commit message: fix aliengo model

File: assets/aliengo_description/xacro/aliengo.urdf (robot description, URDF)
Before this commit: robot aliengo_description, 19 links, 18 joints
Joints:
- joint FL_calf_joint: limit lower=-2.77507351067 upper=-0.645771823238 effort=55 velocity=16 -> lower=0.645771823238 upper=2.77507351067; type continuous -> revolute
- joint FL_hip_joint: limit lower=-1.2217304764 upper=1.2217304764 effort=44 velocity=20 -> lower=-1.4 upper=1.4; type continuous -> revolute
- joint FL_thigh_joint: limit effort=44 velocity=20 -> (none)
- joint FR_calf_joint: limit lower=-2.77507351067 upper=-0.645771823238 effort=55 velocity=16 -> lower=0.645771823238 upper=2.77507351067; type continuous -> revolute
- joint FR_hip_joint: limit lower=-1.2217304764 upper=1.2217304764 effort=44 velocity=20 -> lower=-1.4 upper=1.4; type continuous -> revolute
- joint FR_thigh_joint: limit effort=44 velocity=20 -> (none)
- joint RL_calf_joint: limit lower=-2.77507351067 upper=-0.645771823238 effort=55 velocity=16 -> lower=0.645771823238 upper=2.77507351067; type continuous -> revolute
- joint RL_hip_joint: limit lower=-1.2217304764 upper=1.2217304764 effort=44 velocity=20 -> lower=-1.4 upper=1.4; type continuous -> revolute
- joint RL_thigh_joint: limit effort=44 velocity=20 -> (none)
- joint RR_calf_joint: limit lower=-2.77507351067 upper=-0.645771823238 effort=55 velocity=16 -> lower=0.645771823238 upper=2.77507351067; type continuous -> revolute
- joint RR_hip_joint: limit lower=-1.2217304764 upper=1.2217304764 effort=44 velocity=20 -> lower=-1.4 upper=1.4; type continuous -> revolute
- joint RR_thigh_joint: limit effort=44 velocity=20 -> (none)
