Commit message: add joint pos limit

File: assets/mini_cheetah/mini_cheetah.urdf (robot description, URDF)
Before this commit: robot mini_cheetah, 17 links, 16 joints
Joints:
- joint thigh_fl_to_knee_fl_j: limit (none) -> lower=0.05 upper=2.8; type continuous -> revolute
- joint thigh_fr_to_knee_fr_j: limit (none) -> lower=0.05 upper=2.8; type continuous -> revolute
- joint thigh_hl_to_knee_hl_j: limit (none) -> lower=0.05 upper=2.8; type continuous -> revolute
- joint thigh_hr_to_knee_hr_j: limit (none) -> lower=0.05 upper=2.8; type continuous -> revolute
- joint torso_to_abduct_fl_j: limit (none) -> lower=-1.4 upper=1.4; type continuous -> revolute
- joint torso_to_abduct_fr_j: limit (none) -> lower=-1.4 upper=1.4; type continuous -> revolute
- joint torso_to_abduct_hl_j: limit (none) -> lower=-1.4 upper=1.4; type continuous -> revolute
- joint torso_to_abduct_hr_j: limit (none) -> lower=-1.4 upper=1.4; type continuous -> revolute
