Commit message: minimum modification to make it compatible

File: assets/go1_description/go1.urdf (robot description, URDF)
Before this commit: robot go1, 46 links, 45 joints
Joints:
- joint FL_calf_joint: axis 0 1 0 -> 0 -1 0; type revolute -> continuous
- joint FL_hip_joint: type revolute -> continuous
- joint FL_thigh_joint: axis 0 1 0 -> 0 -1 0; type revolute -> continuous
- joint FR_calf_joint: axis 0 1 0 -> 0 -1 0; type revolute -> continuous
- joint FR_hip_joint: type revolute -> continuous
- joint FR_thigh_joint: axis 0 1 0 -> 0 -1 0; type revolute -> continuous
- joint RL_calf_joint: axis 0 1 0 -> 0 -1 0; type revolute -> continuous
- joint RL_hip_joint: type revolute -> continuous
- joint RL_thigh_joint: axis 0 1 0 -> 0 -1 0; type revolute -> continuous
- joint RR_calf_joint: axis 0 1 0 -> 0 -1 0; type revolute -> continuous
- joint RR_hip_joint: type revolute -> continuous
- joint RR_thigh_joint: axis 0 1 0 -> 0 -1 0; type revolute -> continuous

Commit message: recover calf joint limit

File: assets/go1_description/go1.urdf (robot description, URDF)
Before this commit: robot go1, 46 links, 45 joints
Joints:
- joint FL_calf_joint: limit lower=-2.818 upper=-0.888 effort=35.55 velocity=20.06 -> lower=0.888 upper=2.818 effort=35.55 velocity=20.06; type continuous -> revolute
- joint FR_calf_joint: limit lower=-2.818 upper=-0.888 effort=35.55 velocity=20.06 -> lower=0.888 upper=2.818 effort=35.55 velocity=20.06; type continuous -> revolute
- joint RL_calf_joint: limit lower=-2.818 upper=-0.888 effort=35.55 velocity=20.06 -> lower=0.888 upper=2.818 effort=35.55 velocity=20.06; type continuous -> revolute
- joint RR_calf_joint: limit lower=-2.818 upper=-0.888 effort=35.55 velocity=20.06 -> lower=0.888 upper=2.818 effort=35.55 velocity=20.06; type continuous -> revolute
